Commit message: ++ Collision, forces

File: urdf/quadrotor.urdf.xacro (robot description, xacro)
@@ -7,5 +7,5 @@
   <link name="base_link">
     <inertial>
-      <mass value="1.477" />
+      <mass value="1" />
       <origin xyz="0 0 0" />
       <inertia ixx="0.01152" ixy="0.0" ixz="0.0" iyy="0.01152" iyz="0.0" izz="0.0218" />
@@ -24,4 +24,35 @@
     </collision>
   </link>
+  <gazebo>
+    <plugin name="quadro_sim" filename="libquadro_sim.so">
+      <alwaysOn>true</alwaysOn>
+      <updateRate>0.0</updateRate>
+    </plugin>
+  </gazebo>
+  <gazebo reference="base_link">
+    <sensor name="contact_sensor" type="contact">
+      <always_on>true</always_on>
+      <update_rate>100</update_rate>
+      <contact>
+        <collision>base_link_collision</collision>
+      </contact>
+      <plugin name="gripper_bumper" filename="libgazebo_ros_bumper.so">
+        <bumperTopicName>contact_sensor_state</bumperTopicName>
+        <update_rate>100</update_rate>
+        <always_on>true</always_on>
+        <frameName>gripper</frameName>
+      </plugin>
+    </sensor>
+  </gazebo>
+<!--   <sensor:contact name="contact_sensor">
+    <geom>base_link</geom>
+    <updateRate>10.0</updateRate>
+    <controller:gazebo_ros_bumper name="gazebo_ros_bumper_controller" plugin="libgazebo_ros_bumper.so">
+        <alwaysOn>true</alwaysOn>
+        <updateRate>20.0</updateRate>
+        <bumperTopicName>bumper</bumperTopicName>
+        <interface:bumper name="bumper_iface" />
+    </controller:gazebo_ros_bumper>
+  </sensor:contact> -->
   <!-- Sonar height sensor -->
 <!--   <xacro:sonar_sensor name="sonar_h" parent="base_link" ros_topic="sonar_height" update_rate="40" min_range="0.02" max_range="4.5" field_of_view="${40*pi/180}" ray_count="30">
@@ -34,5 +65,5 @@
     <origin xyz="-0.15 0.0 -0.02" rpy="0 0 ${pi}"/>
   </xacro:sonar_sensor>
-  <xacro:sonar_sensor name="sonar_l" parent="base_link" ros_topic="left" update_rate="40" min_range="0.02" max_range="4.5" field_of_view="${40*pi/180}" ray_count="40">
+  <xacro:sonar_sensor name="sonar_l" parent="base_link" ros_topic="sonar_left" update_rate="40" min_range="0.02" max_range="4.5" field_of_view="${40*pi/180}" ray_count="40">
     <origin xyz="0.0 0.15 -0.02" rpy="0 0 ${90*pi/180}"/>
   </xacro:sonar_sensor>

Commit message: some fixes

File: urdf/quadrotor.urdf.xacro (robot description, xacro)
@@ -1,4 +1,7 @@
 <?xml version="1.0"?>
 <robot name="quadrotor" xmlns:xacro="http://ros.org/wiki/xacro">
+  <xacro:property name="sonar_hor_shift" value="0.15" />
+  <xacro:property name="sonar_ver_shift" value="0.02" />
+  <xacro:property name="sonar_sim_update_rate" value="80" />
   <xacro:include filename="$(find autopilot_simulator)/urdf/sonar_sensor.urdf.xacro" />
   <!-- <xacro:property name="pi" value="3.1415926535897931" /> -->
@@ -28,5 +31,5 @@
     <plugin name="quadro_sim" filename="libquadro_sim.so">
       <alwaysOn>true</alwaysOn>
-      <updateRate>0.0</updateRate>
+      <updateRate>0</updateRate>
     </plugin>
   </gazebo>
@@ -34,5 +37,5 @@
     <sensor name="contact_sensor" type="contact">
       <always_on>true</always_on>
-      <update_rate>10</update_rate>
+      <update_rate>0</update_rate>
       <contact>
         <collision>base_link_collision</collision>
@@ -40,5 +43,4 @@
       <plugin name="gripper_bumper" filename="libgazebo_ros_bumper.so">
         <bumperTopicName>contact_sensor_state</bumperTopicName>
-        <update_rate>10</update_rate>
         <always_on>true</always_on>
         <frameName>gripper</frameName>
@@ -60,15 +62,15 @@
     <origin xyz="0.0 0.0 -0.05" rpy="0 ${90*pi/180} 0"/>
   </xacro:sonar_sensor> -->
-  <xacro:sonar_sensor name="sonar_f" parent="base_link" ros_topic="sonar_front" update_rate="40" min_range="0.02" max_range="4.5" field_of_view="${40*pi/180}" ray_count="40">
-    <origin xyz="0.15 0.0 -0.02" rpy="0 0 0"/>
+  <xacro:sonar_sensor name="sonar_f" parent="base_link" ros_topic="sonar_front" update_rate="${sonar_sim_update_rate}" min_range="0.02" max_range="4.5" field_of_view="${40*pi/180}" ray_count="40">
+    <origin xyz="${sonar_hor_shift} 0.0 -${sonar_ver_shift}" rpy="0 0 0"/>
   </xacro:sonar_sensor>
-  <xacro:sonar_sensor name="sonar_b" parent="base_link" ros_topic="sonar_back" update_rate="40" min_range="0.02" max_range="4.5" field_of_view="${40*pi/180}" ray_count="40">
-    <origin xyz="-0.15 0.0 -0.02" rpy="0 0 ${pi}"/>
+  <xacro:sonar_sensor name="sonar_b" parent="base_link" ros_topic="sonar_back" update_rate="${sonar_sim_update_rate}" min_range="0.02" max_range="4.5" field_of_view="${40*pi/180}" ray_count="40">
+    <origin xyz="-${sonar_hor_shift} 0.0 -${sonar_ver_shift}" rpy="0 0 ${pi}"/>
   </xacro:sonar_sensor>
-  <xacro:sonar_sensor name="sonar_l" parent="base_link" ros_topic="sonar_left" update_rate="40" min_range="0.02" max_range="4.5" field_of_view="${40*pi/180}" ray_count="40">
-    <origin xyz="0.0 0.15 -0.02" rpy="0 0 ${90*pi/180}"/>
+  <xacro:sonar_sensor name="sonar_l" parent="base_link" ros_topic="sonar_left" update_rate="${sonar_sim_update_rate}" min_range="0.02" max_range="4.5" field_of_view="${40*pi/180}" ray_count="40">
+    <origin xyz="0.0 ${sonar_hor_shift} -${sonar_ver_shift}" rpy="0 0 ${90*pi/180}"/>
   </xacro:sonar_sensor>
-  <xacro:sonar_sensor name="sonar_r" parent="base_link" ros_topic="sonar_right" update_rate="40" min_range="0.02" max_range="4.5" field_of_view="${40*pi/180}" ray_count="40">
-    <origin xyz="0.0 -0.15 -0.02" rpy="0 0 ${-90*pi/180}"/>
+  <xacro:sonar_sensor name="sonar_r" parent="base_link" ros_topic="sonar_right" update_rate="${sonar_sim_update_rate}" min_range="0.02" max_range="4.5" field_of_view="${40*pi/180}" ray_count="40">
+    <origin xyz="0.0 -${sonar_hor_shift} -${sonar_ver_shift}" rpy="0 0 ${-90*pi/180}"/>
   </xacro:sonar_sensor>
   <!-- </xacro:macro> -->

Commit message: Some new functions

File: urdf/quadrotor.urdf.xacro (robot description, xacro)
@@ -3,5 +3,5 @@
   <xacro:property name="sonar_hor_shift" value="0.15" />
   <xacro:property name="sonar_ver_shift" value="0.02" />
-  <xacro:property name="sonar_sim_update_rate" value="80" />
+  <xacro:property name="sonar_sim_update_rate" value="100" />
   <xacro:include filename="$(find autopilot_simulator)/urdf/sonar_sensor.urdf.xacro" />
   <!-- <xacro:property name="pi" value="3.1415926535897931" /> -->
@@ -41,21 +41,11 @@
         <collision>base_link_collision</collision>
       </contact>
-      <plugin name="gripper_bumper" filename="libgazebo_ros_bumper.so">
+<!--       <plugin name="gripper_bumper" filename="libgazebo_ros_bumper.so">
         <bumperTopicName>contact_sensor_state</bumperTopicName>
         <always_on>true</always_on>
         <frameName>gripper</frameName>
-      </plugin>
+      </plugin> -->
     </sensor>
   </gazebo>
-<!--   <sensor:contact name="contact_sensor">
-    <geom>base_link</geom>
-    <updateRate>10.0</updateRate>
-    <controller:gazebo_ros_bumper name="gazebo_ros_bumper_controller" plugin="libgazebo_ros_bumper.so">
-        <alwaysOn>true</alwaysOn>
-        <updateRate>20.0</updateRate>
-        <bumperTopicName>bumper</bumperTopicName>
-        <interface:bumper name="bumper_iface" />
-    </controller:gazebo_ros_bumper>
-  </sensor:contact> -->
   <!-- Sonar height sensor -->
 <!--   <xacro:sonar_sensor name="sonar_h" parent="base_link" ros_topic="sonar_height" update_rate="40" min_range="0.02" max_range="4.5" field_of_view="${40*pi/180}" ray_count="30">

File: urdf/sonar_sensor.urdf.xacro (robot description, xacro)
@@ -55,5 +55,4 @@
         </ray>
         <plugin name="gazebo_ros_${name}_controller" filename="libhector_gazebo_ros_sonar.so">
-          <gaussianNoise>0.005</gaussianNoise>
           <topicName>${ros_topic}</topicName>
           <frameId>${name}_link</frameId>
